File: schematics/sbmi/sbmi.sch (KiCad schematic (older format))
At the start: 27 parts, among them J1 Conector JST, J2 Conector de Saídas, J3 Conn_01x04, J4 Recetor IR, J5 Conector Frontal, SW1 Switch, U1 CNY70, U2 CNY70, U3 CNY70, U4 4051, U5 CNY70, U6 CNY70, U7 L7805, U8 L298N

Commit message: dev
Connections:
- net PD5: now also U8.10 (IN3)
- net PD6: now also U8.5 (IN1)
- net MOTOR_DIR-: now reaches U8.14 (OUT4)
- net MOTOR_ESQ-: now reaches U8.3 (OUT2)
- net MOTOR_DIR renamed MOTOR_DIR+
- net MOTOR_ESQ renamed MOTOR_ESQ+
Changed lines of the file:
@@
 	8300 4300 8300 4500
 Text GLabel 9100 4700 2    50   Input ~ 0
-MOTOR_ESQ
+MOTOR_ESQ+
 Text GLabel 9100 5000 2    50   Input ~ 0
-MOTOR_DIR
+MOTOR_DIR+
 Wire Wire Line
 	9100 5000 8900 5000
@@
 Wire Notes Line style solid
 	7000 6500 7000 500
+Text GLabel 7450 4700 0    50   Input ~ 0
+PD6
+Text GLabel 7450 5000 0    50   Input ~ 0
+PD5
+Text GLabel 9100 4800 2    50   Input ~ 0
+MOTOR_ESQ-
+Text GLabel 9100 5100 2    50   Input ~ 0
+MOTOR_DIR-
+Wire Wire Line
+	9100 4800 8900 4800
+Wire Wire Line
+	8900 5100 9100 5100
 $EndSCHEMATC
